Commit message: 0.0.6 24/12/2020 vector_description
Wheels introduced

File: vector_description/urdf/components/camera.urdf.xacro (robot description, xacro)
@@ -1,5 +1,5 @@
 <?xml version="1.0"?>
 <robot xmlns:xacro="http://www.ros.org/wiki/xacro">
-    <xacro:macro name="camera" params="link_name *origin">
+    <macro name="camera" params="link_name *origin">
         <link name="${link_name}"/>
         <joint name="${link_name}_joint" type="fixed">
@@ -8,4 +8,4 @@
             <xacro:insert_block name="origin"/>
         </joint>
-    </xacro:macro>
+    </macro>
 </robot>

File: vector_description/urdf/components/camera.xacro (robot description, xacro)
@@ -1,5 +1,5 @@
 <?xml version="1.0"?>
 <robot xmlns:xacro="http://www.ros.org/wiki/xacro">
-    <xacro:macro name="camera_gazebo">
+    <macro name="camera_gazebo">
         <gazebo reference="camera_link">
             <sensor type="camera" name="vector_camera">
@@ -38,4 +38,4 @@
             </sensor>
         </gazebo>
-    </xacro:macro>
+    </macro>
 </robot>

File: vector_description/urdf/components/drop_sensor.urdf.xacro (robot description, xacro)
@@ -1,5 +1,5 @@
 <?xml version="1.0"?>
 <robot xmlns:xacro="http://www.ros.org/wiki/xacro">
-    <xacro:macro name="drop_sensor" params="link_name *origin">
+    <macro name="drop_sensor" params="link_name *origin">
         <link name="${link_name}"/>
         <joint name="${link_name}_joint" type="fixed">
@@ -8,4 +8,4 @@
             <xacro:insert_block name="origin"/>
         </joint>
-    </xacro:macro>
+    </macro>
 </robot>

File: vector_description/urdf/components/drop_sensor.xacro (robot description, xacro)
@@ -1,5 +1,5 @@
 <?xml version="1.0"?>
 <robot xmlns:xacro="http://www.ros.org/wiki/xacro">
-    <xacro:macro name="drop_sensor_gazebo" params="link_name">
+    <macro name="drop_sensor_gazebo" params="link_name">
         <gazebo reference="${link_name}">
             <sensor type="ray" name="ranger">
@@ -39,4 +39,4 @@
             </sensor>
         </gazebo>
-    </xacro:macro>
+    </macro>
 </robot>

File: vector_description/urdf/components/imu.urdf.xacro (robot description, xacro)
@@ -1,5 +1,5 @@
 <?xml version="1.0"?>
 <robot xmlns:xacro="http://www.ros.org/wiki/xacro">
-    <xacro:macro name="imu_sensor" params="link_name">
+    <macro name="imu_sensor" params="link_name">
         <link name="${link_name}"/>
         <joint name="${link_name}_joint" type="fixed">
@@ -8,4 +8,4 @@
             <origin xyz="0.0 0 0.0" rpy="0 0 0"/>
         </joint>
-    </xacro:macro>
+    </macro>
 </robot>

File: vector_description/urdf/components/imu.xacro (robot description, xacro)
@@ -1,5 +1,5 @@
 <?xml version="1.0"?>
 <robot xmlns:xacro="http://www.ros.org/wiki/xacro">
-    <xacro:macro name="imu_sensor_gazebo">
+    <macro name="imu_sensor_gazebo">
         <gazebo reference="imu">
             <gravity>true</gravity>
@@ -21,4 +21,4 @@
             </sensor>
         </gazebo>
-    </xacro:macro>
+    </macro>
 </robot>

File: vector_description/urdf/vector.urdf.xacro (robot description, xacro)
@@ -5,8 +5,8 @@
     <xacro:include filename="$(find vector_description)/urdf/components/imu.urdf.xacro"/>
     <xacro:include filename="$(find vector_description)/urdf/components/camera.urdf.xacro"/>
+    <xacro:include filename="$(find vector_description)/urdf/components/wheel.urdf.xacro"/>
     <!-- LINKS ===========================  -->
     <!--chassis-->
     <link name="dummy"/>
-    <!--    <link name="imu"/>-->
     <link name="base_link">
         <xacro:box_inertia m="0.06" x="0.073" y="0.043" z="0.061"/>
@@ -22,64 +22,16 @@
         </collision>
     </link>
-    <!--Front left wheel-->
-    <link name="front_left_wheel">
-        <xacro:cylinder_inertia m="0.01" r="0.01314" l="0.0116739"/>
-        <visual>
-            <geometry>
-                <mesh filename="package://vector_description/meshes/flw2.dae"/>
-            </geometry>
-        </visual>
-        <collision>
-            <origin xyz="0 0 0"
-                    rpy="1.57 0 0"/>
-            <geometry>
-                <cylinder radius="${0.026281/2.0}" length="0.0116739"/>
-            </geometry>
-        </collision>
-    </link>
-    <!--Front right wheel  -->
-    <link name="front_right_wheel">
-        <xacro:cylinder_inertia m="0.01" r="0.01314" l="0.0116739"/>
-        <visual>
-            <geometry>
-                <mesh filename="package://vector_description/meshes/flw2.dae"/>
-            </geometry>
-        </visual>
-        <collision>
-            <origin xyz="0 0 0"
-                    rpy="1.57 0 0"/>
-            <geometry>
-                <cylinder radius="${0.026281/2.0}" length="0.0116739"/>
-            </geometry>
-        </collision>
-    </link>
-    <!--Rear left wheel -->
-    <link name="rear_left_wheel">
-        <xacro:cylinder_inertia m="0.01" r="0.008995" l="0.0116739"/>
-        <visual>
-            <geometry>
-                <mesh filename="package://vector_description/meshes/rlw2.dae"/>
-            </geometry>
-        </visual>
-        <collision>
-            <geometry>
-                <mesh filename="package://vector_description/meshes/rlw2.dae"/>
-            </geometry>
-        </collision>
-    </link>
-    <!--Rear right wheel -->
-    <link name="rear_right_wheel">
-        <xacro:cylinder_inertia m="0.01" r="0.008995" l="0.0116739"/>
-        <visual>
-            <geometry>
-                <mesh filename="package://vector_description/meshes/rlw2.dae"/>
-            </geometry>
-        </visual>
-        <collision>
-            <geometry>
-                <mesh filename="package://vector_description/meshes/rlw2.dae"/>
-            </geometry>
-        </collision>
-    </link>
+    <xacro:wheel link_name="front_left_wheel" radius="0.01314" filename="package://vector_description/meshes/flw2.dae">
+        <origin xyz="0.03 0.024 -0.012"/>
+    </xacro:wheel>
+    <xacro:wheel link_name="front_right_wheel" radius="0.01314" filename="package://vector_description/meshes/flw2.dae">
+        <origin xyz="0.03 -0.024 -0.012" rpy="0 0 ${-pi}"/>
+    </xacro:wheel>
+    <xacro:wheel link_name="rear_left_wheel" radius="0.008995" filename="package://vector_description/meshes/rlw2.dae">
+        <origin xyz="-0.017 0.024 -0.0151707"/>
+    </xacro:wheel>
+    <xacro:wheel link_name="rear_right_wheel" radius="0.008995" filename="package://vector_description/meshes/rlw2.dae">
+        <origin xyz="-0.017 -0.024 -0.0151707" rpy="0 0 ${-pi}"/>
+    </xacro:wheel>
     <!-- Head -->
     <link name="head">
@@ -134,5 +86,4 @@
     </link>
     <!-- sensors -->
-    <!--    <link name="camera_link"/>-->
     <xacro:drop_sensor link_name="drop_front_left">
         <origin xyz="0.0351028 0.01 -0.0213898" rpy="0 1.57 0"/>
@@ -155,28 +106,4 @@
         <parent link="dummy"/>
         <child link="base_link"/>
-    </joint>
-    <joint name="base_to_flw" type="continuous">
-        <parent link="base_link"/>
-        <child link="front_left_wheel"/>
-        <origin xyz="0.03 0.024 -0.012"/>
-        <axis xyz="0 1 0"/>
-    </joint>
-    <joint name="base_to_frw" type="continuous">
-        <parent link="base_link"/>
-        <child link="front_right_wheel"/>
-        <origin xyz="0.03 -0.024 -0.012"/>
-        <axis xyz="0 1 0"/>
-    </joint>
-    <joint name="base_to_rlw" type="continuous">
-        <parent link="base_link"/>
-        <child link="rear_left_wheel"/>
-        <origin xyz="-0.017 0.024 -0.0151707"/>
-        <axis xyz="0 1 0"/>
-    </joint>
-    <joint name="base_to_rrw" type="continuous">
-        <parent link="base_link"/>
-        <child link="rear_right_wheel"/>
-        <origin xyz="-0.017 -0.024 -0.0151707"/>
-        <axis xyz="0 1 0"/>
     </joint>
     <joint name="base_to_head" type="revolute">
@@ -207,14 +134,4 @@
         <origin xyz="0.00945088 -0.024 -0.0133211"/>
     </joint>
-<!--    <joint name="head_camera_joint" type="fixed">-->
-<!--        <parent link="head"/>-->
-<!--        <child link="camera_link"/>-->
-<!--        <origin xyz="0.020813 0 -0.0071471" rpy="0 0 0"/>-->
-<!--    </joint>-->
-    <!--    <joint name="imu_joint" type="fixed">-->
-    <!--        <parent link="head"/>-->
-    <!--        <child link="imu"/>-->
-    <!--        <origin xyz="0.0 0 0.0" rpy="0 0 0"/>-->
-    <!--    </joint>-->
     <gazebo reference="rear_right_wheel">
         <mu1>0.5</mu1>
@@ -261,30 +178,4 @@
         </actuator>
     </transmission>
-    <!-- ROS Control plugin for Gazebo -->
-    <gazebo>
-        <plugin name="gazebo_ros_control" filename="libgazebo_ros_control.so">
-            <robotNamespace>/vector</robotNamespace>
-            <legacyModeNS>true</legacyModeNS>
-        </plugin>
-    </gazebo>
-    <gazebo>
-        <plugin name="skid_steer_drive_controller" filename="libgazebo_ros_skid_steer_drive.so">
-            <updateRate>25.0</updateRate>
-            <robotNamespace>/</robotNamespace>
-            <leftFrontJoint>base_to_flw</leftFrontJoint>
-            <rightFrontJoint>base_to_frw</rightFrontJoint>
-            <leftRearJoint>base_to_rlw</leftRearJoint>
-            <rightRearJoint>base_to_rrw</rightRearJoint>
-            <wheelSeparation>0.048</wheelSeparation>
-            <wheelDiameter>0.026281</wheelDiameter>
-            <robotBaseFrame>base_link</robotBaseFrame>
-            <torque>20</torque>
-            <topicName>cmd_vel</topicName>
-            <commandTopic>cmd_vel</commandTopic>
-            <odometryTopic>odom</odometryTopic>
-            <odometryFrame>odom</odometryFrame>
-            <broadcastTF>1</broadcastTF>
-        </plugin>
-    </gazebo>
     <!-- components -->
     <xacro:include filename="$(find vector_description)/urdf/vector.gazebo"/>
