Commit message: 0.0.5 23/12/2020 vector_description
Camera introduced

File: vector_description/urdf/vector.urdf.xacro (robot description, xacro)
@@ -4,4 +4,5 @@
     <xacro:include filename="$(find vector_description)/urdf/components/drop_sensor.urdf.xacro"/>
     <xacro:include filename="$(find vector_description)/urdf/components/imu.urdf.xacro"/>
+    <xacro:include filename="$(find vector_description)/urdf/components/camera.urdf.xacro"/>
     <!-- LINKS ===========================  -->
     <!--chassis-->
@@ -133,5 +134,5 @@
     </link>
     <!-- sensors -->
-    <link name="camera_link"/>
+    <!--    <link name="camera_link"/>-->
     <xacro:drop_sensor link_name="drop_front_left">
         <origin xyz="0.0351028 0.01 -0.0213898" rpy="0 1.57 0"/>
@@ -147,4 +148,7 @@
     </xacro:drop_sensor>
     <xacro:imu_sensor link_name="imu"/>
+    <xacro:camera link_name="camera">
+        <origin xyz="0.020813 0 -0.0071471" rpy="0 0 0"/>
+    </xacro:camera>
     <!-- JOINTS ====================================-->
     <joint name="dummy_joint" type="fixed">
@@ -203,9 +207,9 @@
         <origin xyz="0.00945088 -0.024 -0.0133211"/>
     </joint>
-    <joint name="head_camera_joint" type="fixed">
-        <parent link="head"/>
-        <child link="camera_link"/>
-        <origin xyz="0.020813 0 -0.0071471" rpy="0 0 0"/>
-    </joint>
+<!--    <joint name="head_camera_joint" type="fixed">-->
+<!--        <parent link="head"/>-->
+<!--        <child link="camera_link"/>-->
+<!--        <origin xyz="0.020813 0 -0.0071471" rpy="0 0 0"/>-->
+<!--    </joint>-->
     <!--    <joint name="imu_joint" type="fixed">-->
     <!--        <parent link="head"/>-->
@@ -283,40 +287,4 @@
         </plugin>
     </gazebo>
-    <gazebo reference="camera_link">
-        <sensor type="camera" name="cozmo_camera">
-            <update_rate>10.0</update_rate>
-            <camera name="headcamera">
-                <horizontal_fov>1.3962634</horizontal_fov>
-                <image>
-                    <width>1280</width>
-                    <height>720</height>
-                    <format>R8G8B8</format>
-                </image>
-                <clip>
-                    <near>0.01</near>
-                    <far>100</far>
-                </clip>
-                <noise>
-                    <type>gaussian</type>
-                    <mean>0.0</mean>
-                    <stddev>0.007</stddev>
-                </noise>
-            </camera>
-            <plugin name="camera_controller" filename="libgazebo_ros_camera.so">
-                <alwaysOn>true</alwaysOn>
-                <updateRate>25.0</updateRate>
-                <cameraName>camera</cameraName>
-                <imageTopicName>image</imageTopicName>
-                <cameraInfoTopicName>camera_info</cameraInfoTopicName>
-                <frameName>camera_link</frameName>
-                <hackBaseline>0.07</hackBaseline>
-                <distortionK1>0.0</distortionK1>
-                <distortionK2>0.0</distortionK2>
-                <distortionK3>0.0</distortionK3>
-                <distortionT1>0.0</distortionT1>
-                <distortionT2>0.0</distortionT2>
-            </plugin>
-        </sensor>
-    </gazebo>
     <!-- components -->
     <xacro:include filename="$(find vector_description)/urdf/vector.gazebo"/>

Commit message: 0.0.7 24/12/2020 vector_description
Belts introduced

File: vector_description/urdf/vector.urdf.xacro (robot description, xacro)
@@ -6,4 +6,5 @@
     <xacro:include filename="$(find vector_description)/urdf/components/camera.urdf.xacro"/>
     <xacro:include filename="$(find vector_description)/urdf/components/wheel.urdf.xacro"/>
+    <xacro:include filename="$(find vector_description)/urdf/components/belt.urdf.xacro"/>
     <!-- LINKS ===========================  -->
     <!--chassis-->
@@ -34,4 +35,10 @@
         <origin xyz="-0.017 -0.024 -0.0151707" rpy="0 0 ${-pi}"/>
     </xacro:wheel>
+    <xacro:belt link_name="left_belt" filename="package://vector_description/meshes/cozmo_belt.dae">
+        <origin xyz="0.00945088 0.024 -0.0133211"/>
+    </xacro:belt>
+    <xacro:belt link_name="right_belt" filename="package://vector_description/meshes/cozmo_belt.dae">
+        <origin xyz="0.00945088 -0.024 -0.0133211"/>
+    </xacro:belt>
     <!-- Head -->
     <link name="head">
@@ -61,27 +68,4 @@
             </geometry>
         </collision>
-    </link>
-    <!-- Belts -->
-    <link name="left_belt">
-        <inertial>
-            <mass value="0.0001"/>
-            <inertia ixx="0.000001" ixy="0" ixz="0" iyy="0.000001" iyz="0" izz="0.0000001"/>
-        </inertial>
-        <visual>
-            <geometry>
-                <mesh filename="package://vector_description/meshes/cozmo_belt.dae"/>
-            </geometry>
-        </visual>
-    </link>
-    <link name="right_belt">
-        <inertial>
-            <mass value="0.0001"/>
-            <inertia ixx="0.000001" ixy="0" ixz="0" iyy="0.000001" iyz="0" izz="0.0000001"/>
-        </inertial>
-        <visual>
-            <geometry>
-                <mesh filename="package://vector_description/meshes/cozmo_belt.dae"/>
-            </geometry>
-        </visual>
     </link>
     <!-- sensors -->
@@ -123,14 +107,4 @@
         <dynamics damping="0.0" friction="0.1"/>
         <axis xyz="0 1 0"/>
-    </joint>
-    <joint name="wheel_left_belt" type="fixed">
-        <parent link="base_link"/>
-        <child link="left_belt"/>
-        <origin xyz="0.00945088 0.024 -0.0133211"/>
-    </joint>
-    <joint name="wheel_right_belt" type="fixed">
-        <parent link="base_link"/>
-        <child link="right_belt"/>
-        <origin xyz="0.00945088 -0.024 -0.0133211"/>
     </joint>
     <gazebo reference="rear_right_wheel">

Commit message: 0.0.8 24/12/2020 vector_description
Meshes added

File: vector_description/urdf/vector.urdf.xacro (robot description, xacro)
@@ -7,7 +7,9 @@
     <xacro:include filename="$(find vector_description)/urdf/components/wheel.urdf.xacro"/>
     <xacro:include filename="$(find vector_description)/urdf/components/belt.urdf.xacro"/>
-    <!-- LINKS ===========================  -->
-    <!--chassis-->
     <link name="dummy"/>
+    <joint name="dummy_joint" type="fixed">
+        <parent link="dummy"/>
+        <child link="base_link"/>
+    </joint>
     <link name="base_link">
         <xacro:box_inertia m="0.06" x="0.073" y="0.043" z="0.061"/>
@@ -20,4 +22,49 @@
             <geometry>
                 <mesh filename="package://vector_description/meshes/vector_body.dae"/>
+            </geometry>
+        </collision>
+    </link>
+    <joint name="base_to_head" type="revolute">
+        <parent link="base_link"/>
+        <child link="head"/>
+        <origin xyz="0.0174507 0 0.022003"/>
+        <limit lower="-0.52" upper="0.17" effort="100" velocity="10"/>
+        <!-- Dampning break the model, keep it 0.0 -->
+        <dynamics damping="0.0" friction="0.1"/>
+        <axis xyz="0 1 0"/>
+    </joint>
+    <!-- Head -->
+    <link name="head">
+        <xacro:box_inertia m="0.01" x="0.036" y="0.038" z="0.041"/>
+        <visual>
+            <geometry>
+                <mesh filename="package://vector_description/meshes/vector_head.dae"/>
+            </geometry>
+        </visual>
+        <collision>
+            <geometry>
+                <mesh filename="package://vector_description/meshes/vector_head.dae"/>
+            </geometry>
+        </collision>
+    </link>
+    <joint name="base_to_lift" type="revolute">
+        <parent link="base_link"/>
+        <child link="full_lift"/>
+        <origin xyz="-0.005 0 0.013"/>
+        <limit lower="-0.8" upper="0" effort="5" velocity="10"/>
+        <dynamics damping="0.0" friction="0.1"/>
+        <axis xyz="0 1 0"/>
+    </joint>
+    <!-- lifter -->
+    <link name="full_lift">
+        <xacro:box_inertia m="0.01" x="0.081" y="0.058" z="0.050"/>
+        <visual>
+            <geometry>
+                <mesh filename="package://vector_description/meshes/vector_lift.dae"/>
+            </geometry>
+        </visual>
+        <collision>
+            <geometry>
+                <mesh filename="package://vector_description/meshes/vector_lift.dae"/>
             </geometry>
         </collision>
@@ -41,32 +88,4 @@
         <origin xyz="0.00945088 -0.024 -0.0133211"/>
     </xacro:belt>
-    <!-- Head -->
-    <link name="head">
-        <xacro:box_inertia m="0.01" x="0.036" y="0.038" z="0.041"/>
-        <visual>
-            <geometry>
-                <mesh filename="package://vector_description/meshes/vector_head.dae"/>
-            </geometry>
-        </visual>
-        <collision>
-            <geometry>
-                <mesh filename="package://vector_description/meshes/vector_head.dae"/>
-            </geometry>
-        </collision>
-    </link>
-    <!-- lifter -->
-    <link name="full_lift">
-        <xacro:box_inertia m="0.01" x="0.081" y="0.058" z="0.050"/>
-        <visual>
-            <geometry>
-                <mesh filename="package://vector_description/meshes/vector_lift.dae"/>
-            </geometry>
-        </visual>
-        <collision>
-            <geometry>
-                <mesh filename="package://vector_description/meshes/vector_lift.dae"/>
-            </geometry>
-        </collision>
-    </link>
     <!-- sensors -->
     <xacro:drop_sensor link_name="drop_front_left">
@@ -86,26 +105,4 @@
         <origin xyz="0.020813 0 -0.0071471" rpy="0 0 0"/>
     </xacro:camera>
-    <!-- JOINTS ====================================-->
-    <joint name="dummy_joint" type="fixed">
-        <parent link="dummy"/>
-        <child link="base_link"/>
-    </joint>
-    <joint name="base_to_head" type="revolute">
-        <parent link="base_link"/>
-        <child link="head"/>
-        <origin xyz="0.0174507 0 0.022003"/>
-        <limit lower="-0.52" upper="0.17" effort="100" velocity="10"/>
-        <!-- Dampning break the model, keep it 0.0 -->
-        <dynamics damping="0.0" friction="0.1"/>
-        <axis xyz="0 1 0"/>
-    </joint>
-    <joint name="base_to_lift" type="revolute">
-        <parent link="base_link"/>
-        <child link="full_lift"/>
-        <origin xyz="-0.005 0 0.013"/>
-        <limit lower="-0.8" upper="0" effort="5" velocity="10"/>
-        <dynamics damping="0.0" friction="0.1"/>
-        <axis xyz="0 1 0"/>
-    </joint>
     <gazebo reference="rear_right_wheel">
         <mu1>0.5</mu1>
