Commit message: 0.0.4 23/12/2020 vector_description
Drop sensors and IMU introduced

File: vector_description/urdf/common/inertia.xacro (robot description, xacro)
@@ -2,5 +2,5 @@
 <robot xmlns:xacro="http://www.ros.org/wiki/xacro">
     <macro name="cylinder_inertia" params="m r l">
-        <mass value="${m}" />
+        <mass value="${m}"/>
         <inertia ixx="${m*(3*r*r+l*l)/12}" ixy="0" ixz="0"
                  iyy="${m*(3*r*r+l*l)/12}" iyz="0"
@@ -8,5 +8,5 @@
     </macro>
     <macro name="box_inertia" params="m x y z">
-        <mass value="${m}" />
+        <mass value="${m}"/>
         <inertia ixx="${m*(y*y+z*z)/12}" ixy="0" ixz="0"
                  iyy="${m*(x*x+z*z)/12}" iyz="0"
@@ -14,14 +14,8 @@
     </macro>
     <macro name="sphere_inertia" params="m r">
-        <mass value="${m}" />
+        <mass value="${m}"/>
         <inertia ixx="${2*m*r*r/5}" ixy="0" ixz="0"
                  iyy="${2*m*r*r/5}" iyz="0"
                  izz="${2*m*r*r/5}"/>
     </macro>
-    <macro name="box_inertia_default" params="m">
-        <inertial>
-            <mass value="${m}"/>
-            <inertia ixx="0.000001" ixy="0" ixz="0" iyy="0.000001" iyz="0" izz="0.0000001"/>
-        </inertial>
-    </macro>
 </robot>

File: vector_description/urdf/components/imu.xacro (robot description, xacro)
@@ -1,5 +1,5 @@
 <?xml version="1.0"?>
 <robot xmlns:xacro="http://www.ros.org/wiki/xacro">
-    <xacro:macro name="imu">
+    <xacro:macro name="imu_sensor_gazebo">
         <gazebo reference="imu">
             <gravity>true</gravity>

File: vector_description/urdf/vector.urdf.xacro (robot description, xacro)
@@ -2,9 +2,10 @@
 <robot name="vector" xmlns:xacro="http://www.ros.org/wiki/xacro">
     <xacro:include filename="$(find vector_description)/urdf/common/inertia.xacro"/>
+    <xacro:include filename="$(find vector_description)/urdf/components/drop_sensor.urdf.xacro"/>
+    <xacro:include filename="$(find vector_description)/urdf/components/imu.urdf.xacro"/>
     <!-- LINKS ===========================  -->
     <!--chassis-->
-    <link name="dummy">
-    </link>
-    <link name="imu"/>
+    <link name="dummy"/>
+    <!--    <link name="imu"/>-->
     <link name="base_link">
         <xacro:box_inertia m="0.06" x="0.073" y="0.043" z="0.061"/>
@@ -131,10 +132,19 @@
         </visual>
     </link>
-    <!-- sensors links -->
+    <!-- sensors -->
     <link name="camera_link"/>
-    <link name="drop_ir_fl"/>
-    <link name="drop_ir_fr"/>
-    <link name="drop_ir_rl"/>
-    <link name="drop_ir_rr"/>
+    <xacro:drop_sensor link_name="drop_front_left">
+        <origin xyz="0.0351028 0.01 -0.0213898" rpy="0 1.57 0"/>
+    </xacro:drop_sensor>
+    <xacro:drop_sensor link_name="drop_front_right">
+        <origin xyz="0.0351028 -0.01 -0.0213898" rpy="0 1.57 0"/>
+    </xacro:drop_sensor>
+    <xacro:drop_sensor link_name="drop_rear_left">
+        <origin xyz="-0.02 0.01 -0.0213898" rpy="0 1.57 0"/>
+    </xacro:drop_sensor>
+    <xacro:drop_sensor link_name="drop_rear_right">
+        <origin xyz="-0.02 -0.01 -0.0213898" rpy="0 1.57 0"/>
+    </xacro:drop_sensor>
+    <xacro:imu_sensor link_name="imu"/>
     <!-- JOINTS ====================================-->
     <joint name="dummy_joint" type="fixed">
@@ -198,29 +208,9 @@
         <origin xyz="0.020813 0 -0.0071471" rpy="0 0 0"/>
     </joint>
-    <joint name="drop_ir_fl_joint" type="fixed">
-        <parent link="base_link"/>
-        <child link="drop_ir_fl"/>
-        <origin xyz="0.0351028 0.01 -0.0213898" rpy="0 1.57 0"/>
-    </joint>
-    <joint name="drop_ir_fr_joint" type="fixed">
-        <parent link="base_link"/>
-        <child link="drop_ir_fr"/>
-        <origin xyz="0.0351028 -0.01 -0.0213898" rpy="0 1.57 0"/>
-    </joint>
-    <joint name="drop_ir_rl_joint" type="fixed">
-        <parent link="base_link"/>
-        <child link="drop_ir_rl"/>
-        <origin xyz="-0.02 0.01 -0.0213898" rpy="0 1.57 0"/>
-    </joint>
-    <joint name="drop_ir_rr_joint" type="fixed">
-        <parent link="base_link"/>
-        <child link="drop_ir_rr"/>
-        <origin xyz="-0.02 -0.01 -0.0213898" rpy="0 1.57 0"/>
-    </joint>
-    <joint name="imu_joint" type="fixed">
-        <parent link="head"/>
-        <child link="imu"/>
-        <origin xyz="0.0 0 0.0" rpy="0 0 0"/>
-    </joint>
+    <!--    <joint name="imu_joint" type="fixed">-->
+    <!--        <parent link="head"/>-->
+    <!--        <child link="imu"/>-->
+    <!--        <origin xyz="0.0 0 0.0" rpy="0 0 0"/>-->
+    <!--    </joint>-->
     <gazebo reference="rear_right_wheel">
         <mu1>0.5</mu1>
@@ -329,152 +319,4 @@
         </sensor>
     </gazebo>
-    <gazebo reference="drop_ir_fl">
-        <sensor type="ray" name="TeraRanger">
-            <pose>0 0 0 0 0 0</pose>
-            <visualize>true</visualize>
-            <update_rate>50</update_rate>
-            <ray>
-                <scan>
-                    <horizontal>
-                        <samples>10</samples>
-                        <resolution>1</resolution>
-                        <min_angle>-0.14835</min_angle>
-                        <max_angle>0.14835</max_angle>
-                    </horizontal>
-                    <vertical>
-                        <samples>10</samples>
-                        <resolution>1</resolution>
-                        <min_angle>-0.14835</min_angle>
-                        <max_angle>0.14835</max_angle>
-                    </vertical>
-                </scan>
-                <range>
-                    <min>0.01</min>
-                    <max>2</max>
-                    <resolution>0.02</resolution>
-                </range>
-            </ray>
-            <plugin filename="libgazebo_ros_range.so" name="gazebo_ros_range">
-                <gaussianNoise>0.005</gaussianNoise>
-                <alwaysOn>true</alwaysOn>
-                <updateRate>50</updateRate>
-                <topicName>drop_sensor_fl</topicName>
-                <frameName>drop_ir_fl</frameName>
-                <radiation>INFRARED</radiation>
-                <fov>0.2967</fov>
-            </plugin>
-        </sensor>
-    </gazebo>
-    <gazebo reference="drop_ir_fr">
-        <sensor type="ray" name="TeraRanger">
-            <pose>0 0 0 0 0 0</pose>
-            <visualize>true</visualize>
-            <update_rate>50</update_rate>
-            <ray>
-                <scan>
-                    <horizontal>
-                        <samples>10</samples>
-                        <resolution>1</resolution>
-                        <min_angle>-0.14835</min_angle>
-                        <max_angle>0.14835</max_angle>
-                    </horizontal>
-                    <vertical>
-                        <samples>10</samples>
-                        <resolution>1</resolution>
-                        <min_angle>-0.14835</min_angle>
-                        <max_angle>0.14835</max_angle>
-                    </vertical>
-                </scan>
-                <range>
-                    <min>0.01</min>
-                    <max>2</max>
-                    <resolution>0.02</resolution>
-                </range>
-            </ray>
-            <plugin filename="libgazebo_ros_range.so" name="gazebo_ros_range">
-                <gaussianNoise>0.005</gaussianNoise>
-                <alwaysOn>true</alwaysOn>
-                <updateRate>50</updateRate>
-                <topicName>drop_sensor_fr</topicName>
-                <frameName>drop_ir_fr</frameName>
-                <radiation>INFRARED</radiation>
-                <fov>0.2967</fov>
-            </plugin>
-        </sensor>
-    </gazebo>
-    <gazebo reference="drop_ir_rl">
-        <sensor type="ray" name="TeraRanger">
-            <pose>0 0 0 0 0 0</pose>
-            <visualize>true</visualize>
-            <update_rate>50</update_rate>
-            <ray>
-                <scan>
-                    <horizontal>
-                        <samples>10</samples>
-                        <resolution>1</resolution>
-                        <min_angle>-0.14835</min_angle>
-                        <max_angle>0.14835</max_angle>
-                    </horizontal>
-                    <vertical>
-                        <samples>10</samples>
-                        <resolution>1</resolution>
-                        <min_angle>-0.14835</min_angle>
-                        <max_angle>0.14835</max_angle>
-                    </vertical>
-                </scan>
-                <range>
-                    <min>0.01</min>
-                    <max>2</max>
-                    <resolution>0.02</resolution>
-                </range>
-            </ray>
-            <plugin filename="libgazebo_ros_range.so" name="gazebo_ros_range">
-                <gaussianNoise>0.005</gaussianNoise>
-                <alwaysOn>true</alwaysOn>
-                <updateRate>50</updateRate>
-                <topicName>drop_sensor_rl</topicName>
-                <frameName>drop_ir_rl</frameName>
-                <radiation>INFRARED</radiation>
-                <fov>0.2967</fov>
-            </plugin>
-        </sensor>
-    </gazebo>
-    <gazebo reference="drop_ir_rr">
-        <sensor type="ray" name="TeraRanger">
-            <pose>0 0 0 0 0 0</pose>
-            <visualize>true</visualize>
-            <update_rate>50</update_rate>
-            <ray>
-                <scan>
-                    <horizontal>
-                        <samples>10</samples>
-                        <resolution>1</resolution>
-                        <min_angle>-0.14835</min_angle>
-                        <max_angle>0.14835</max_angle>
-                    </horizontal>
-                    <vertical>
-                        <samples>10</samples>
-                        <resolution>1</resolution>
-                        <min_angle>-0.14835</min_angle>
-                        <max_angle>0.14835</max_angle>
-                    </vertical>
-                </scan>
-                <range>
-                    <min>0.01</min>
-                    <max>2</max>
-                    <resolution>0.02</resolution>
-                </range>
-            </ray>
-            <plugin filename="libgazebo_ros_range.so" name="gazebo_ros_range">
-                <gaussianNoise>0.005</gaussianNoise>
-                <alwaysOn>true</alwaysOn>
-                <updateRate>50</updateRate>
-                <topicName>drop_sensor_rr</topicName>
-                <frameName>drop_ir_rr</frameName>
-                <radiation>INFRARED</radiation>
-                <fov>0.2967</fov>
-            </plugin>
-        </sensor>
-    </gazebo>
     <!-- components -->
     <xacro:include filename="$(find vector_description)/urdf/vector.gazebo"/>
