Commit message: 0.0.9 16/01/2021 vector_description
xacro/macro housekeeping and mass added to inertia tags for fixing simulation

File: vector_description/urdf/common/inertia.xacro (robot description, xacro)
@@ -1,21 +1,12 @@
 <?xml version="1.0"?>
 <robot xmlns:xacro="http://www.ros.org/wiki/xacro">
-    <macro name="cylinder_inertia" params="m r l">
-        <mass value="${m}"/>
-        <inertia ixx="${m*(3*r*r+l*l)/12}" ixy="0" ixz="0"
-                 iyy="${m*(3*r*r+l*l)/12}" iyz="0"
-                 izz="${m*r*r/2}"/>
-    </macro>
-    <macro name="box_inertia" params="m x y z">
-        <mass value="${m}"/>
-        <inertia ixx="${m*(y*y+z*z)/12}" ixy="0" ixz="0"
-                 iyy="${m*(x*x+z*z)/12}" iyz="0"
-                 izz="${m*(x*x+z*z)/12}"/>
-    </macro>
-    <macro name="sphere_inertia" params="m r">
-        <mass value="${m}"/>
-        <inertia ixx="${2*m*r*r/5}" ixy="0" ixz="0"
-                 iyy="${2*m*r*r/5}" iyz="0"
-                 izz="${2*m*r*r/5}"/>
-    </macro>
+	<macro name="cylinder_inertia" params="m r l">
+		<inertia ixx="${m*(3*r*r+l*l)/12}" ixy="0" ixz="0" iyy="${m*(3*r*r+l*l)/12}" iyz="0" izz="${m*r*r/2}" />
+	</macro>
+	<macro name="box_inertia" params="m x y z">
+		<inertia ixx="${m*(y*y+z*z)/12}" ixy="0" ixz="0" iyy="${m*(x*x+z*z)/12}" iyz="0" izz="${m*(x*x+z*z)/12}" />
+	</macro>
+	<macro name="sphere_inertia" params="m r">
+		<inertia ixx="${2*m*r*r/5}" ixy="0" ixz="0" iyy="${2*m*r*r/5}" iyz="0" izz="${2*m*r*r/5}" />
+	</macro>
 </robot>

File: vector_description/urdf/components/belt.urdf.xacro (robot description, xacro)
@@ -16,5 +16,5 @@
             <parent link="base_link"/>
             <child link="${link_name}"/>
-            <xacro:insert_block name="origin"/>
+            <insert_block name="origin"/>
         </joint>
     </macro>

File: vector_description/urdf/components/camera.urdf.xacro (robot description, xacro)
@@ -6,5 +6,5 @@
             <parent link="head"/>
             <child link="${link_name}"/>
-            <xacro:insert_block name="origin"/>
+            <insert_block name="origin"/>
         </joint>
     </macro>

File: vector_description/urdf/components/drop_sensor.urdf.xacro (robot description, xacro)
@@ -6,5 +6,5 @@
             <parent link="base_link"/>
             <child link="${link_name}"/>
-            <xacro:insert_block name="origin"/>
+            <insert_block name="origin"/>
         </joint>
     </macro>

File: vector_description/urdf/components/wheel.urdf.xacro (robot description, xacro)
@@ -22,5 +22,5 @@
                 </geometry>
                 <mass value="0.01"/>
-                <xacro:cylinder_inertia m="0.01" r="${radius}" l="0.01167"/>
+                <cylinder_inertia m="0.01" r="${radius}" l="0.01167"/>
             </inertial>
         </link>
@@ -28,5 +28,5 @@
             <parent link="base_link"/>
             <child link="${link_name}"/>
-            <xacro:insert_block name="origin"/>
+            <insert_block name="origin"/>
             <axis xyz="0 1 0"/>
         </joint>

File: vector_description/urdf/vector.urdf.xacro (robot description, xacro)
@@ -1,17 +1,25 @@
 <?xml version="1.0"?>
 <robot name="vector" xmlns:xacro="http://www.ros.org/wiki/xacro">
-    <xacro:include filename="$(find vector_description)/urdf/common/inertia.xacro"/>
-    <xacro:include filename="$(find vector_description)/urdf/components/drop_sensor.urdf.xacro"/>
-    <xacro:include filename="$(find vector_description)/urdf/components/imu.urdf.xacro"/>
-    <xacro:include filename="$(find vector_description)/urdf/components/camera.urdf.xacro"/>
-    <xacro:include filename="$(find vector_description)/urdf/components/wheel.urdf.xacro"/>
-    <xacro:include filename="$(find vector_description)/urdf/components/belt.urdf.xacro"/>
-    <link name="dummy"/>
-    <joint name="dummy_joint" type="fixed">
-        <parent link="dummy"/>
+    <include filename="$(find vector_description)/urdf/common/inertia.xacro"/>
+    <include filename="$(find vector_description)/urdf/components/drop_sensor.urdf.xacro"/>
+    <include filename="$(find vector_description)/urdf/components/imu.urdf.xacro"/>
+    <include filename="$(find vector_description)/urdf/components/camera.urdf.xacro"/>
+    <include filename="$(find vector_description)/urdf/components/wheel.urdf.xacro"/>
+    <include filename="$(find vector_description)/urdf/components/belt.urdf.xacro"/>
+    <link name="base_footprint"/>
+    <joint name="base_footprint_joint" type="fixed">
+        <origin rpy="0 0 0" xyz="0 0 0.027"/>
+        <parent link="base_footprint"/>
         <child link="base_link"/>
     </joint>
     <link name="base_link">
-        <xacro:box_inertia m="0.06" x="0.073" y="0.043" z="0.061"/>
+        <inertial>
+            <origin rpy="0 0 0" xyz="0.0075 0.0 -0.01"/>
+            <geometry>
+                <box size="0.073 0.043 0.061"/>
+            </geometry>
+            <mass value="0.16"/>
+            <box_inertia m="0.16" x="0.073" y="0.043" z="0.061"/>
+        </inertial>
         <visual>
             <geometry>
@@ -20,9 +28,19 @@
         </visual>
         <collision>
-            <geometry>
-                <mesh filename="package://vector_description/meshes/vector_body.dae"/>
+            <origin rpy="0 0 0" xyz="0.0075 0.0 -0.01"/>
+            <geometry>
+                <box size="0.07 0.03 0.01"/>
             </geometry>
         </collision>
     </link>
+    <gazebo reference="base_link">
+        <selfCollide>
+            true
+        </selfCollide>
+        <mu1 value="200.0"/>
+        <mu2 value="100.0"/>
+        <kp value="10000000.0"/>
+        <kd value="1.0"/>
+    </gazebo>
     <joint name="base_to_head" type="revolute">
         <parent link="base_link"/>
@@ -36,5 +54,11 @@
     <!-- Head -->
     <link name="head">
-        <xacro:box_inertia m="0.01" x="0.036" y="0.038" z="0.041"/>
+        <inertial>
+            <geometry>
+                <sphere radius="0.02"/>
+            </geometry>
+            <mass value="0.03"/>
+            <sphere_inertia m="0.03" r="0.02"/>
+        </inertial>
         <visual>
             <geometry>
@@ -44,8 +68,14 @@
         <collision>
             <geometry>
-                <mesh filename="package://vector_description/meshes/vector_head.dae"/>
+                <sphere radius="0.02"/>
             </geometry>
         </collision>
     </link>
+    <gazebo reference="head">
+        <mu1 value="200.0"/>
+        <mu2 value="100.0"/>
+        <kp value="10000000.0"/>
+        <kd value="1.0"/>
+    </gazebo>
     <joint name="base_to_lift" type="revolute">
         <parent link="base_link"/>
@@ -58,5 +88,12 @@
     <!-- lifter -->
     <link name="full_lift">
-        <xacro:box_inertia m="0.01" x="0.081" y="0.058" z="0.050"/>
+        <inertial>
+            <origin rpy="0 0 0" xyz="0.062 0.0 -0.015"/>
+            <geometry>
+                <box size="0.0075 0.05 0.025"/>
+            </geometry>
+            <mass value="0.05"/>
+            <box_inertia m="0.05" x="0.0075" y="0.05" z="0.025"/>
+        </inertial>
         <visual>
             <geometry>
@@ -65,44 +102,51 @@
         </visual>
         <collision>
-            <geometry>
-                <mesh filename="package://vector_description/meshes/vector_lift.dae"/>
+            <origin rpy="0 0 0" xyz="0.062 0.0 -0.015"/>
+            <geometry>
+                <box size="0.0075 0.05 0.025"/>
             </geometry>
         </collision>
     </link>
-    <xacro:wheel link_name="front_left_wheel" radius="0.01314" filename="package://vector_description/meshes/flw2.dae">
+    <gazebo reference="full_lift">
+        <mu1 value="200.0"/>
+        <mu2 value="100.0"/>
+        <kp value="10000000.0"/>
+        <kd value="1.0"/>
+    </gazebo>
+    <wheel link_name="front_left_wheel" radius="0.01314" filename="package://vector_description/meshes/flw2.dae">
         <origin xyz="0.03 0.024 -0.012"/>
-    </xacro:wheel>
-    <xacro:wheel link_name="front_right_wheel" radius="0.01314" filename="package://vector_description/meshes/flw2.dae">
+    </wheel>
+    <wheel link_name="front_right_wheel" radius="0.01314" filename="package://vector_description/meshes/flw2.dae">
         <origin xyz="0.03 -0.024 -0.012" rpy="0 0 ${-pi}"/>
-    </xacro:wheel>
-    <xacro:wheel link_name="rear_left_wheel" radius="0.008995" filename="package://vector_description/meshes/rlw2.dae">
+    </wheel>
+    <wheel link_name="rear_left_wheel" radius="0.008995" filename="package://vector_description/meshes/rlw2.dae">
         <origin xyz="-0.017 0.024 -0.0151707"/>
-    </xacro:wheel>
-    <xacro:wheel link_name="rear_right_wheel" radius="0.008995" filename="package://vector_description/meshes/rlw2.dae">
+    </wheel>
+    <wheel link_name="rear_right_wheel" radius="0.008995" filename="package://vector_description/meshes/rlw2.dae">
         <origin xyz="-0.017 -0.024 -0.0151707" rpy="0 0 ${-pi}"/>
-    </xacro:wheel>
-    <xacro:belt link_name="left_belt" filename="package://vector_description/meshes/cozmo_belt.dae">
+    </wheel>
+    <belt link_name="left_belt" filename="package://vector_description/meshes/cozmo_belt.dae">
         <origin xyz="0.00945088 0.024 -0.0133211"/>
-    </xacro:belt>
-    <xacro:belt link_name="right_belt" filename="package://vector_description/meshes/cozmo_belt.dae">
+    </belt>
+    <belt link_name="right_belt" filename="package://vector_description/meshes/cozmo_belt.dae">
         <origin xyz="0.00945088 -0.024 -0.0133211"/>
-    </xacro:belt>
+    </belt>
     <!-- sensors -->
-    <xacro:drop_sensor link_name="drop_front_left">
+    <drop_sensor link_name="drop_front_left">
         <origin xyz="0.0351028 0.01 -0.0213898" rpy="0 1.57 0"/>
-    </xacro:drop_sensor>
-    <xacro:drop_sensor link_name="drop_front_right">
+    </drop_sensor>
+    <drop_sensor link_name="drop_front_right">
         <origin xyz="0.0351028 -0.01 -0.0213898" rpy="0 1.57 0"/>
-    </xacro:drop_sensor>
-    <xacro:drop_sensor link_name="drop_rear_left">
+    </drop_sensor>
+    <drop_sensor link_name="drop_rear_left">
         <origin xyz="-0.02 0.01 -0.0213898" rpy="0 1.57 0"/>
-    </xacro:drop_sensor>
-    <xacro:drop_sensor link_name="drop_rear_right">
+    </drop_sensor>
+    <drop_sensor link_name="drop_rear_right">
         <origin xyz="-0.02 -0.01 -0.0213898" rpy="0 1.57 0"/>
-    </xacro:drop_sensor>
-    <xacro:imu_sensor link_name="imu"/>
-    <xacro:camera link_name="camera">
+    </drop_sensor>
+    <imu_sensor link_name="imu"/>
+    <camera link_name="camera">
         <origin xyz="0.020813 0 -0.0071471" rpy="0 0 0"/>
-    </xacro:camera>
+    </camera>
     <gazebo reference="rear_right_wheel">
         <mu1>0.5</mu1>
@@ -121,33 +165,42 @@
         <mu2>100000</mu2>
     </gazebo>
-    <gazebo reference="head">
-        <kp>1000000000.0</kp>
-        <kd>1000000000.0</kd>
-        <mu1>10.0</mu1>
-        <mu2>10.0</mu2>
-        <self_collide>0</self_collide>
-    </gazebo>
     <!-- Transmissions for joints -->
     <transmission name="base_to_head_trans">
-        <type>transmission_interface/SimpleTransmission</type>
+        <type>
+            transmission_interface/SimpleTransmission
+        </type>
         <joint name="base_to_head">
-            <hardwareInterface>hardware_interface/EffortJointInterface</hardwareInterface>
+            <hardwareInterface>
+                hardware_interface/EffortJointInterface
+            </hardwareInterface>
         </joint>
         <actuator name="base_to_headMotor">
-            <hardwareInterface>hardware_interface/EffortJointInterface</hardwareInterface>
-            <mechanicalReduction>1</mechanicalReduction>
+            <hardwareInterface>
+                hardware_interface/EffortJointInterface
+            </hardwareInterface>
+            <mechanicalReduction>
+                1
+            </mechanicalReduction>
         </actuator>
     </transmission>
     <transmission name="base_to_lift_trans">
-        <type>transmission_interface/SimpleTransmission</type>
+        <type>
+            transmission_interface/SimpleTransmission
+        </type>
         <joint name="base_to_lift">
-            <hardwareInterface>hardware_interface/EffortJointInterface</hardwareInterface>
+            <hardwareInterface>
+                hardware_interface/EffortJointInterface
+            </hardwareInterface>
         </joint>
         <actuator name="base_to_liftMotor">
-            <hardwareInterface>hardware_interface/EffortJointInterface</hardwareInterface>
-            <mechanicalReduction>1</mechanicalReduction>
+            <hardwareInterface>
+                hardware_interface/EffortJointInterface
+            </hardwareInterface>
+            <mechanicalReduction>
+                1
+            </mechanicalReduction>
         </actuator>
     </transmission>
     <!-- components -->
-    <xacro:include filename="$(find vector_description)/urdf/vector.gazebo"/>
+    <include filename="$(find vector_description)/urdf/vector.gazebo"/>
 </robot>
